File: dc2025_badge/dc2025_badge.kicad_pcb (KiCad board)
At the start: 2 copper layers, 244 x 93 mm, 489 parts, among them J1 USB_C_Receptacle_USB2.0_16P, J2 Conn_ARM_JTAG_SWD_10, Q1 AO3401A, U1 TPS3808DBV, U2 STM32L053R8Tx, U3 IS31FL3731-QF, U4 ST25R3916-AQWT, U5 XC6206P332MR, U6 XC6206P332MR, Y1 27.12MHz

Commit message: 0603 leds added, prototype version finished
Parts:
- added G***: LOGO, logo:hg_logo, B.Cu at (84.1, 116.9)
- added G***: LOGO, logo:hg_logo_text, B.Cu at (81.0, 122.9)
- added R11: 100k, Resistor_SMD:R_0402_1005Metric, F.Cu at (69.7, 102.9)
- added REF**: OSHW-Logo2_14.6x12mm_SilkScreen, Symbol:OSHW-Logo2_14.6x12mm_SilkScreen, B.Cu at (44.4, 64.0)
- AE1: value Antenna_Dipole -> Antenna
- D10, D100, D101, D102, D103, D104, D105, D106, D107, D108, D109, D11, D110, D111, D112, D113, D114, D115, D116, D117, D118, D119, D12, D120, D121, D122, D123, D124, D125, D126, D127, D128, D129, D13, D130, D131, D132, D133, D134, D135, D136, D137, D138, D139, D14, D140, D141, D142, D143, D144, D145, D146, D147, D148, D149, D15, D150, D151, D152, D153, D154, D155, D156, D157, D158, D159, D16, D160, D161, D162, D163, D164, D165, D166, D167, D168, D169, D17, D170, D171, D172, D173, D174, D175, D176, D177, D178, D179, D18, D180, D181, D182, D183, D184, D185, D186, D187, D188, D189, D19, D190, D191, D192, D193, D194, D195, D196, D197, D198, D199, D2, D20, D200, D201, D202, D21, D22, D23, D24, D25, D26, D27, D28, D29, D3, D30, D31, D32, D33, D34, D35, D36, D37, D38, D39, D4, D40, D41, D42, D43, D44, D45, D46, D47, D48, D49, D5, D50, D51, D52, D53, D54, D55, D56, D57, D58, D59, D6, D60, D61, D62, D63, D64, D65, D66, D67, D68, D69, D7, D70, D71, D72, D73, D74, D75, D76, D77, D78, D79, D8, D80, D81, D82, D83, D84, D85, D86, D87, D88, D89, D9, D90, D91, D92, D93, D94, D95, D96, D97, D98, D99: footprint LED_SMD:LED_0402_1005Metric -> LED_SMD:LED_0603_1608Metric
- H10, H7, H8, H9: value MountingHole -> CoverMountingHole
- H3, H4, H5, H6: value Cover mount -> Cover nut
- moved D164 0.31 mm to (75.6, 73.5)
- moved D46 0.25 mm to (92.2, 73.5)
- moved R159 0.17 mm to (125.1, 71.1)
- moved R133 0.17 mm to (57.6, 71.1)
- moved R92 0.17 mm to (40.8, 71.1)
- moved R64 0.08 mm to (91.1, 71.2)
- moved R15 0.07 mm to (74.3, 71.2)
Connections:
- S1 pad SH1: (no net) -> GND
- S1 pad SH2: (no net) -> GND
- S1 pad SH3: (no net) -> GND
- S1 pad SH4: (no net) -> GND
Routing:
- net /LEDs/CA6: track 252.6 -> 262.7 mm
- net /LEDs/CA7: track 228.9 -> 237.9 mm
- net /LEDs/CA8: track 225.6 -> 232.6 mm
- net /LEDs/CA4: track 244.3 -> 251.2 mm
- net /LEDs/CA2: track 278.7 -> 285.1 mm, vias 12 -> 14
- net /LEDs/CB4: track 95.0 -> 100.3 mm
- net /LEDs/CB1: track 72.6 -> 77.5 mm, vias 7 -> 9
- net /LEDs/CA1: track 232.6 -> 236.1 mm
- net /LEDs/CA3: track 256.5 -> 260.0 mm
- net /LEDs/CA5: track 260.5 -> 263.5 mm
- net /LEDs/CB7: track 65.5 -> 67.7 mm
- net /LEDs/CB2: track 97.4 -> 99.4 mm, vias 8 -> 10
- net /LEDs/CB3: track 85.5 -> 87.1 mm
- net VDD: track 167.6 -> 169.0 mm
- net /NFC/BSS: track 51.1 -> 52.3 mm
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Other:
- board text added: "30TH OPEN SYSTEM DAYS / CROATIAN LINUX USERS' CONFERENCE"
- board text added: "5765277265206E6F20737472616E6765 727320746F206C6F76652C20596F7520 6B6E6F77207468652072756C65732061 6E6420736F20646F20492C2041206675 6C6C20636F6D6D69746D656E74277320 776861742049276D207468696E6B696E 67206F662C20596F7520776F756C646E 27742067657420746869732066726F6D 20616E79206F74686572206775792E"
- board text added: "DORS/CLUC 2025"
- board text added: "made by: hyperglitch.com"
