File: dc2025_badge/nfc.kicad_sch (KiCad schematic)
At the start: 37 parts, among them U4 ST25R3916-AQWT, Y1 27.12MHz

Commit message: 0603 leds added, prototype version finished
Parts:
- added R11: 100k, Resistor_SMD:R_0402_1005Metric, symbol Device:R
- AE1: value Antenna_Dipole -> Antenna
- C12, C13, C35, C38: MPN (none) -> CL05C100JB5NNNC; Manufacturer (none) -> Samsung Electro-Mechanics
- C14, C24, C25, C26, C27, C34: MPN (none) -> CL10A225KO8NNNC; Manufacturer (none) -> Samsung Electro-Mechanics
- C30, C33: MPN (none) -> 0402B221K500NT; Manufacturer (none) -> FH (Guangdong Fenghua Advanced Tech)
- C31, C32: MPN (none) -> 0402B681K500NT; Manufacturer (none) -> FH (Guangdong Fenghua Advanced Tech)
- C36, C37, C39, C40: MPN (none) -> 0402B151K500NT; Manufacturer (none) -> FH (Guangdong Fenghua Advanced Tech)
- L1, L2: MPN (none) -> LQB15NNR27K10D; Manufacturer (none) -> Murata Electronics
- R175, R176: MPN (none) -> WR04X2R0JTL; Manufacturer (none) -> Walsin Tech Corp
- U4: MPN (none) -> ST25R3916-AQWT; Manufacturer (none) -> STMicroelectronics
Connections:
- net BSS: now also R11.2
- net VDD: now also R11.1
Other:
- note removed: "?"
- moved on the sheet: AE1, C12, C13, C14, C15, C16, C17, C18, C19, C20, C21, C22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
