File: dc2025_badge/production/main-20250504-2/dc2025_badge.kicad_pcb (KiCad board)
At the start: 2 copper layers, 112.9 x 98 mm, 482 parts, among them J1 USB_C_Receptacle_USB2.0_16P, J2 Conn_ARM_JTAG_SWD_10, Q1 AO3401A, U1 TPS3808DBV, U2 STM32L073RBT6, U3 IS31FL3731-QF, U4 ST25R3916-AQWT, U5 XC6206P332MR, U6 XC6206P332MR, Y1 27.12MHz

Commit message: hardware added production version
Parts:
- added H10: CoverMountingHole, MountingHole:MountingHole_3.2mm_M3_DIN965, F.Cu at (251.1, 98.7)
- added H7: CoverMountingHole, MountingHole:MountingHole_3.2mm_M3_DIN965, F.Cu at (182.1, 130.0)
- added H8: CoverMountingHole, MountingHole:MountingHole_3.2mm_M3_DIN965, F.Cu at (179.1, 49.0)
- added H9: CoverMountingHole, MountingHole:MountingHole_3.2mm_M3_DIN965, F.Cu at (258.1, 49.0)
Routing:
- net (no net): track 0.00 -> 1661.0 mm
Other:
- board size 112.9 x 98 mm -> 244 x 98 mm
- board text added: "5765277265206E6F20737472616E6765 727320746F206C6F76652C20596F7520 6B6E6F77207468652072756C65732061 6E6420736F20646F20492C2041206675 6C6C20636F6D6D69746D656E74277320 776861742049276D207468696E6B696E 67206F662C20596F7520776F756C646E 27742067657420746869732066726F6D 20616E79206F74686572206775792E"
- board text added: "DORS/CLUC 2025"
